File: Hardware/PCB/Motor_driver/Motor_driver.kicad_sch (KiCad schematic)
At the start: 67 parts, among them IC1 A89307KETSR-J, IC2 STM32L412KBT6, IC3 AZ1117CH2-3.3TRG1, J1 ENCODER, J2 USB_C, J4 Debug, SW1 SW_Nidec_CAS-120A1, SW2 SW_Nidec_CAS-120A1

Commit message: Premier jet schematic PCB moteur
Parts:
- removed R11, R12, R13, R14: 10k, symbol Device:R
- removed SW1, SW2: SW_Nidec_CAS-120A1, Button_Switch_SMD:Nidec_Copal_CAS-120A, symbol Switch:SW_Nidec_CAS-120A1
- added J3: PAD_MOTEUR, Custom:Solder Pad x3, symbol Connector:Conn_01x03_Pin
- added J5, J6, J7, J8: Conn_01x01_Pin, MountingHole:MountingHole_3.2mm_M3_Pad_TopBottom, symbol Connector:Conn_01x01_Pin
- added R17, R18: 10k, Resistor_SMD:R_0603_1608Metric, symbol Device:R
- added S3: 418121270802, SamacSys_Parts:418121270802, symbol SamacSys_Parts:418121270802
- added TP11: 24V, TestPoint:TestPoint_Pad_D1.5mm, symbol Connector:TestPoint
- added TP12: 5V, TestPoint:TestPoint_Pad_D1.5mm, symbol Connector:TestPoint
- added TP13: 3.3V, TestPoint:TestPoint_Pad_D1.5mm, symbol Connector:TestPoint
- added U1: ~, Custom:452406020024, symbol Custom:switch_452406020024
- L1: footprint (none) -> SamacSys_Parts:WE-MAPI_3020
- Oscillator1: footprint (none) -> Custom:Oscillator 7x5mm
- R1, R10, R15, R16, R2, R3, R4, R5, R6, R7, R8, R9: footprint (none) -> Resistor_SMD:R_0603_1608Metric
- SQJ746ELP1, SQJ746ELP2, SQJ746ELP3: footprint (none) -> Package_SO:PowerPAK_SO-8_Dual
- TP1: value TestPoint -> SDA; footprint (none) -> TestPoint:TestPoint_Pad_D1.5mm
- TP10: value TestPoint -> BRAKE; footprint (none) -> TestPoint:TestPoint_Pad_D1.5mm
- TP2: value TestPoint -> SCL; footprint (none) -> TestPoint:TestPoint_Pad_D1.5mm
- TP3: value TestPoint -> RX; footprint (none) -> TestPoint:TestPoint_Pad_D1.5mm
- TP4: value TestPoint -> TX; footprint (none) -> TestPoint:TestPoint_Pad_D1.5mm
- TP5: value TestPoint -> GATE C; footprint (none) -> TestPoint:TestPoint_Pad_D1.5mm
- TP6: value TestPoint -> GATE B; footprint (none) -> TestPoint:TestPoint_Pad_D1.5mm
- TP7: value TestPoint -> GATE A; footprint (none) -> TestPoint:TestPoint_Pad_D1.5mm
- TP8: value TestPoint -> PWM; footprint (none) -> TestPoint:TestPoint_Pad_D1.5mm
- TP9: value TestPoint -> DIR; footprint (none) -> TestPoint:TestPoint_Pad_D1.5mm
- XT60: footprint (none) -> Connector_AMASS:AMASS_XT60-F_1x02_P7.20mm_Vertical
- renumbered IC3 to PS2
Connections:
- net VBB is gone; now on net +24V: SQJ746ELP1.1 (S1), SQJ746ELP2.1 (S1), SQJ746ELP3.1 (S1), XT60.1 (Pin_1)
- net +24V: now also TP11.1
- net +3.3V: now also R17.1, R18.1, TP13.1
- net +5V: now also TP12.1
- net GND: now also J5.1 (Pin_1), J6.1 (Pin_1), J7.1 (Pin_1), J8.1 (Pin_1)
- net PWM: now also IC2.18 (PA8), U1.6; no longer IC1.24 (SPD)
- net SA: now also J3.3 (Pin_3)
- net SB: now also J3.2 (Pin_2)
- net SC: now also J3.1 (Pin_1)
- net SCL: now also U1.4
- net SDA: now also U1.1; no longer IC1.27 (FG)
- net at IC2.14 (PB0): now also S3.3 (2)
- net at IC2.15 (PB1): now also S3.4 (1)
- net D+: no longer names the net of IC2.22 (PA12)
- net D- renamed PA11
- net PA11: now also U1.3
- new net: R18.2, S3.1
- new net: R17.2, S3.2
- new net FG: IC1.27 (FG), U1.2
- new net SPD: IC1.24 (SPD), U1.5
- no-connect marks 14 -> 16
Other:
- note added: "DATA"
- note added: "MOUNTING HOLES"
- note added: "POWER"
- note added: "Switch pour passer du mode I2C a PWM"
- moved on the sheet: C10, C14, C15, C16, C17, C18, C19, C20, C5, C6, D1, D4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
