File: Hardware/PCB/Motor_driver/arm_bridge.kicad_sch (KiCad schematic)
At the start: 9 parts

Commit message: clean schematic
Other:
- moved on the sheet: C23, R12, R14, R23, R24, SQJ746ELP1, TP14, TP15, TP16
