File: Hardware/PCB/Motor_driver/arm_bridge.kicad_sch (KiCad schematic)
At the start: 9 parts

Commit message: Pcb moteur routé
Connections:
- net +24V: now also SQJ746ELP1.5 (D1); no longer SQJ746ELP1.6 (D1)
- net Sx: now also SQJ746ELP1.6 (D2); no longer SQJ746ELP1.5 (D2)
Changed lines of the file:
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@@
 			)
 		)
-		(property "Datasheet" ""
+		(property "Datasheet" "https://www.vishay.com/docs/62293/sqj746elp.pdf"
 			(at 34.29 46.99 0)
 			(effects
