File: Hardware/TMC262_Stepper_Driver/TMC262_Stepper_Driver.kicad_sch (KiCad schematic)
At the start: 90 parts, among them J1 Conn_01x02, J2 Conn_01x04, J4 629722000214, J6 629712010214, Q1 SQJ504EP, Q2 SQJ504EP, Q3 SQJ504EP, Q4 SQJ504EP, SW5 SW_Push, SW6 SW_Push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

Commit message: update footprint
Parts:
- C10, C12, C13, C27, C3, C7: footprint (none) -> Capacitor_SMD:C_0402_1005Metric
- C11: footprint (none) -> Capacitor_SMD:C_0805_2012Metric
- C28, C29: footprint (none) -> Capacitor_SMD:C_2220_5750Metric
- C6: footprint (none) -> Capacitor_SMD:C_0603_1608Metric
- D2, D3: footprint Diode_SMD:D_SMA -> (none)
- J2: footprint (none) -> Connector_JST:JST_XH_B4B-XH-A_1x04_P2.50mm_Vertical
- R1, R16, R17, R2, R3: footprint (none) -> Resistor_SMD:R_0402_1005Metric
- SW5, SW6, SW7, SW8: footprint SamacSys_Parts:430152043826 -> (none)
- U1: footprint Package_TO_SOT_SMD:SOT-223 -> (none)
Changed lines of the file:
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@@
 		(at 81.28 209.55)
 	)
+	(bus_entry
+		(at 203.2 104.14)
+		(size 2.54 2.54)
+		(stroke
+			(width 0)
+			(type default)
+		)
+	)
+	(bus_entry
+		(at 170.18 100.33)
+		(size 2.54 2.54)
+		(stroke
+			(width 0)
+			(type default)
+		)
+	)
 	(wire
 		(pts
@@
 			)
 		)
-		(property "Footprint" ""
+		(property "Footprint" "Capacitor_SMD:C_0402_1005Metric"
 			(at 196.85 151.13 0)
 			(effects
@@
 			)
 		)
-		(property "Footprint" ""
+		(property "Footprint" "Capacitor_SMD:C_0402_1005Metric"
 			(at 331.47 185.42 0)
 			(effects
@@
 			)
 		)
-		(property "Footprint" ""
+		(property "Footprint" "Capacitor_SMD:C_0402_1005Metric"
 			(at 331.47 241.3 0)
 			(effects
@@
 			)
 		)
-		(property "Footprint" ""
+		(property "Footprint" "Connector_JST:JST_XH_B4B-XH-A_1x04_P2.50mm_Vertical"
 			(at 375.92 193.04 0)
 			(effects
@@
 			)
 		)
-		(property "Footprint" ""
+		(property "Footprint" "Capacitor_SMD:C_0603_1608Metric"
 			(at 207.01 151.13 0)
 			(effects
@@
 			)
 		)
-		(property "Footprint" ""
+		(property "Footprint" "Resistor_SMD:R_0402_1005Metric"
 			(at 180.34 62.23 0)
 			(effects
@@
 			)
 		)
-		(property "Footprint" ""
+		(property "Footprint" "Capacitor_SMD:C_0805_2012Metric"
 			(at 182.88 152.4 0)
 			(effects
@@
 			)
 		)
-		(property "Footprint" ""
+		(property "Footprint" "Resistor_SMD:R_0402_1005Metric"
 			(at 201.93 187.96 0)
 			(effects
@@
 			)
 		)
-		(property "Footprint" ""
+		(property "Footprint" "Capacitor_SMD:C_2220_5750Metric"
 			(at 368.3 220.98 0)
 			(effects
@@
 			)
 		)
-		(property "Footprint" "SamacSys_Parts:430152043826"
+		(property "Footprint" ""
 			(at 392.43 39.37 0)
 			(effects
@@
 			)
 		)
-		(property "Footprint" ""
+		(property "Footprint" "Resistor_SMD:R_0402_1005Metric"
 			(at 304.8 181.61 0)
 			(effects
@@
 			)
 		)
-		(property "Footprint" ""
+		(property "Footprint" "Capacitor_SMD:C_2220_5750Metric"
 			(at 368.3 166.37 0)
 			(effects
@@
 			)
 		)
-		(property "Footprint" ""
+		(property "Footprint" "Capacitor_SMD:C_0402_1005Metric"
 			(at 161.29 152.4 0)
 			(effects
@@
 			)
 		)
-		(property "Footprint" "Package_TO_SOT_SMD:SOT-223"
+		(property "Footprint" ""
 			(at 140.97 35.56 0)
 			(effects
@@
 			)
 		)
-		(property "Footprint" ""
+		(property "Footprint" "Capacitor_SMD:C_0402_1005Metric"
 			(at 242.57 151.13 0)
 			(effects
@@
 			)
 		)
-		(property "Footprint" "SamacSys_Parts:430152043826"
+		(property "Footprint" ""
 			(at 382.27 63.5 0)
 			(effects
@@
 			)
 		)
-		(property "Footprint" ""
+		(property "Footprint" "Resistor_SMD:R_0402_1005Metric"
 			(at 304.8 237.49 0)
 			(effects
@@
 			)
 		)
-		(property "Footprint" ""
+		(property "Footprint" "Capacitor_SMD:C_0402_1005Metric"
 			(at 172.72 152.4 0)
 			(effects
@@
 			)
 		)
-		(property "Footprint" "SamacSys_Parts:430152043826"
+		(property "Footprint" ""
 			(at 364.49 72.39 0)
 			(effects
@@
 			)
 		)
-		(property "Footprint" "Diode_SMD:D_SMA"
+		(property "Footprint" ""
 			(at 63.5 83.82 0)
 			(effects
@@
 			)
 		)
-		(property "Footprint" "Diode_SMD:D_SMA"
+		(property "Footprint" ""
 			(at 63.5 91.44 0)
 			(effects
@@
 			)
 		)
-		(property "Footprint" ""
+		(property "Footprint" "Resistor_SMD:R_0402_1005Metric"
 			(at 252.73 226.06 0)
 			(effects
@@
 			)
 		)
-		(property "Footprint" "SamacSys_Parts:430152043826"
+		(property "Footprint" ""
 			(at 364.49 39.37 0)
 			(effects
