File: Hardware/TMC262_Stepper_Driver/TMC262_Stepper_Driver-backups/TMC262_Stepper_Driver-2025-04-05_184558/TMC262_Stepper_Driver.kicad_sch (KiCad schematic)
At the start: 103 parts, among them J1 Conn_01x04, J3 629722000214, J4 Conn_01x02, J5 Conn_01x04, J6 Conn_01x05, Q1 SQJ504EP, Q2 SQJ504EP, Q3 SQJ504EP, Q4 SQJ504EP, SW1 SW_Push, SW2 SW_Push, SW3 SW_Push, SW4 SW_Push, SW5 SW_Push, U1 AZ1117-3.3, U3 STM32G431CBUx, U4 TMC262, U5 USBLC6-2SC6

Commit message: stepper done
Parts:
- removed C31: 1u, Capacitor_SMD:C_0402_1005Metric, symbol Device:C_Small
- removed J6: Conn_01x05, Connector_JST:JST_PH_B5B-PH-K_1x05_P2.00mm_Vertical, symbol Connector_Generic:Conn_01x05
- removed JP1: SolderJumper_3_Open, Jumper:SolderJumper-3_P2.0mm_Open_TrianglePad1.0x1.5mm, symbol Jumper:SolderJumper_3_Open
- added C16: 100n, Capacitor_SMD:C_0402_1005Metric, symbol Device:C_Small
- added D12: WS2812B, LED_SMD:LED_WS2812B_PLCC4_5.0x5.0mm_P3.2mm, symbol LED:WS2812B
- J4: renamed from J5; footprint Connector_JST:JST_PH_B4B-PH-K_1x04_P2.00mm_Vertical -> Connector_JST:JST_EH_B4B-EH-A_1x04_P2.50mm_Vertical
- Q1, Q4: footprint Maker_librairy:SQJ504EP -> Maker:SQJ504EP
- Q2: renamed from Q3; footprint Maker_librairy:SQJ504EP -> Maker:SQJ504EP
- Q3: renamed from Q2; footprint Maker_librairy:SQJ504EP -> Maker:SQJ504EP
- renumbered C7 to C1, C25 to C10, C20 to C11, C21 to C12, C15 to C13, C22 to C14, C16 to C15, C1 to C17, C2 to C18, C3 to C19, C8 to C2, C4 to C20, C5 to C21, C6 to C22, C29 to C23, C27 to C24, C9 to C25, C18 to C26, C26 to C27, C10 to C29, C14 to C3, C19 to C30, C30 to C4, C11 to C5, C12 to C6, C13 to C7, C23 to C8, C24 to C9, D4 to D1, D1 to D10, D2 to D11, D11 to D2, D12 to D3, D5 to D4, D6 to D5, D7 to D6, D8 to D7, D9 to D8, D10 to D9, J4 to J1, J1 to J5, R7 to R1, R16 to R10, R17 to R11, R8 to R12, R22 to R13, R25 to R14, R26 to R15, R18 to R16, R27 to R17, R28 to R18, R5 to R2, R29 to R20, R20 to R21, R30 to R22, R21 to R23, R3 to R24, R10 to R25, R1 to R26, R9 to R27, R4 to R28, R2 to R29, R6 to R3, R11 to R30, R12 to R4, R23 to R5, R24 to R6, R13 to R7, R14 to R8, R15 to R9, SW4 to SW2, SW2 to SW3, SW3 to SW4, U2 to U1, U1 to U2, U5 to U3, U3 to U5
Connections:
- net +24V: now also J1.1 (Pin_1); no longer J1.2 (Pin_2)
- net +5V: now also C16.1, D12.1 (VDD)
- net GND: now also J1.2 (Pin_2), C16.2, D12.3 (VSS); no longer J1.1 (Pin_1), U1.10 (AGND), U1.13 (PGND)
- net at D11.2 (DOUT): now also D12.4 (DIN)
Other:
- moved on the sheet: J1
